File: small_wind_turbine/KiCAD/small_wind_turbine/small_wind_turbine.kicad_pcb (KiCad board)
At the start: 2 copper layers, 83 parts, among them J1 Conn_01x03_Male, J2 Conn_01x03_Male, J3 Conn_01x03_Male, K1 G5LE-1, Q1 Q_NMOS_GDS, SW1 SW_Push_SPDT, U10 AZ1117-5.0, U2 UC2844A, U3 LTC4440ES6, U4 Opamp_Quad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

Commit message: start layout (1)
Parts:
- added TP1: TestPoint_2Pole, small_wind_turbine:Oscilloscope_Test_Point, F.Cu at (249.0, 111.9)
- added TP10: TestPoint_2Pole, small_wind_turbine:Oscilloscope_Test_Point, F.Cu at (222.0, 122.0)
- added TP11: TestPoint_2Pole, small_wind_turbine:Oscilloscope_Test_Point, F.Cu at (235.5, 127.0)
- added TP2: TestPoint_2Pole, small_wind_turbine:Oscilloscope_Test_Point, F.Cu at (222.0, 111.9)
- added TP3: TestPoint_2Pole, small_wind_turbine:Oscilloscope_Test_Point, F.Cu at (235.5, 122.0)
- added TP4: TestPoint_2Pole, small_wind_turbine:Oscilloscope_Test_Point, F.Cu at (235.5, 117.0)
- added TP5: TestPoint_2Pole, small_wind_turbine:Oscilloscope_Test_Point, F.Cu at (235.5, 111.9)
- added TP6: TestPoint_2Pole, small_wind_turbine:Oscilloscope_Test_Point, F.Cu at (249.0, 122.0)
- added TP7: TestPoint_2Pole, small_wind_turbine:Oscilloscope_Test_Point, F.Cu at (222.0, 117.0)
- added TP8: TestPoint_2Pole, small_wind_turbine:Oscilloscope_Test_Point, F.Cu at (249.0, 117.0)
- added TP9: TestPoint_2Pole, small_wind_turbine:Oscilloscope_Test_Point, F.Cu at (222.0, 127.0)
- Dbs1, Dbuck1: footprint Package_TO_SOT_SMD:TO-277A -> small_wind_turbine:TO-277A
- K1: moved to B.Cu
- moved Dbs1 139.0 mm to (24.9, 101.0)
- moved Cbs1 129.6 mm to (31.0, 102.0)
- moved U3 114.8 mm to (35.1, 91.0)
- moved Dbuck1 92.1 mm to (52.0, 103.0)
- moved C1 60.7 mm to (167.3, 111.7)
- moved C2 60.7 mm to (174.2, 127.5)
- moved J2 60.7 mm to (177.5, 104.3)
- moved J3 60.7 mm to (172.8, 104.3)
- moved R14 60.7 mm to (174.0, 133.4)
- moved U10 60.7 mm to (165.6, 106.1)
- moved U5 60.7 mm to (174.2, 114.9)
- moved U7 60.7 mm to (165.0, 127.8)
- moved C10 60.7 mm to (169.8, 127.5)
- moved C12 60.7 mm to (184.6, 120.2)
- moved C13 60.7 mm to (188.4, 114.2)
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Routing:
- net Net-(D3-Pad2): track 17.4 -> 0.00 mm
- net Net-(D5-Pad2): track 17.3 -> 0.00 mm
- net Net-(D1-Pad2): track 17.3 -> 0.00 mm

Commit message: wip layout (2)
Parts:
- Cbs1: footprint Capacitor_SMD:C_0805_2012Metric -> Capacitor_THT:CP_Radial_D8.0mm_P3.50mm
- moved TP1 189.9 mm to (66.0, 61.0)
- moved R12 113.8 mm to (96.4, 61.2)
- moved Dbuck1 84.6 mm to (124.0, 58.7), turned to -90 degrees
- moved Cbs1 71.5 mm to (93.3, 67.0)
- moved Dbs1 70.1 mm to (90.0, 75.0), turned to 180 degrees
- moved U3 62.5 mm to (95.2, 74.0), turned to 90 degrees
- moved U2 53.0 mm to (96.0, 81.0), turned to 90 degrees
- moved K1 17.3 mm to (98.0, 56.3), turned to 0 degrees
- moved Q1 7.21 mm to (90.0, 62.0), turned to 0 degrees
- moved Cinput1 4.00 mm to (123.0, 52.0)
- moved Jres1 3.53 mm to (125.7, 39.5)
- moved Lbuck1 1.41 mm to (114.0, 75.0)
- moved Qbuck1 1.05 mm to (110.9, 60.0)
- moved Cbuck1 1.00 mm to (109.0, 96.0)
- moved Rsh1 1.00 mm to (102.0, 91.5)
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
Commit message: wip layout (3)
Parts:
- moved C15 133.7 mm to (65.0, 73.0)
- moved C11 129.3 mm to (74.0, 76.0)
- moved C16 128.1 mm to (65.0, 75.0)
- moved U6 126.6 mm to (56.0, 72.0)
- moved C10 122.1 mm to (61.0, 72.0), turned to -90 degrees
- moved C14 119.0 mm to (65.0, 71.0)
- moved U5 111.2 mm to (71.5, 72.1)
- moved U10 103.7 mm to (65.0, 81.0), turned to -90 degrees
- moved Jbat1 80.3 mm to (50.3, 63.0), turned to 90 degrees
- moved Rsh2 54.1 mm to (57.0, 68.0), turned to 180 degrees
- moved Cbuck1 53.6 mm to (65.0, 65.3), turned to 90 degrees
- moved Q1 38.4 mm to (114.0, 32.0), turned to -90 degrees
- moved Rsh1 37.3 mm to (73.0, 68.0), turned to 180 degrees
- moved Lbuck1 29.1 mm to (88.0, 62.0), turned to 180 degrees
- moved TP1 29.0 mm to (66.0, 32.0)
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
Commit message: wip layout (4)
Parts:
- moved C18 159.4 mm to (54.0, 93.2), turned to 90 degrees
- moved C17 153.2 mm to (56.0, 93.2), turned to 90 degrees
- moved R6 149.0 mm to (57.7, 80.2), turned to 180 degrees
- moved R5 147.7 mm to (64.9, 74.4), turned to 180 degrees
- moved C9 147.0 mm to (55.3, 89.5), turned to 90 degrees
- moved R3 146.1 mm to (57.7, 78.2)
- moved R4 144.0 mm to (64.9, 72.2)
- moved R8 132.9 mm to (67.5, 84.2)
- moved U9 132.0 mm to (58.4, 89.5)
- moved R2 131.4 mm to (57.7, 76.2), turned to 180 degrees
- moved R7 129.1 mm to (57.7, 82.2), turned to 180 degrees
- moved U4 126.8 mm to (64.6, 79.2), turned to -90 degrees
- moved R9 124.7 mm to (67.5, 86.2)
- moved C8 123.6 mm to (53.3, 89.5), turned to 90 degrees
- moved J3 122.8 mm to (52.0, 82.5), turned to 180 degrees
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Connections:
- R2 pad 1: Net-(U4-Pad2) -> Net-(U4-Pad6)
- R3 pad 2: Net-(U4-Pad2) -> Net-(U4-Pad6)
- TP9 pad 1: Net-(U4-Pad3) -> Net-(TP9-Pad1)
- U4 pad 1: Net-(R6-Pad2) -> Net-(J2-Pad2)
- U4 pad 10: Net-(R6-Pad1) -> unconnected-(U4-Pad10)
- U4 pad 12: Net-(R4-Pad2) -> Net-(R6-Pad1)
- U4 pad 13: Net-(J2-Pad2) -> Net-(R8-Pad1)
- U4 pad 14: Net-(J2-Pad2) -> Net-(R8-Pad2)
- U4 pad 2: Net-(U4-Pad2) -> Net-(J2-Pad2)
- U4 pad 3: Net-(U4-Pad3) -> Net-(R4-Pad2)
- U4 pad 5: unconnected-(U4-Pad5) -> Net-(TP9-Pad1)
- U4 pad 6: unconnected-(U4-Pad6) -> Net-(U4-Pad6)
- U4 pad 7: unconnected-(U4-Pad7) -> Net-(R6-Pad2)
- U4 pad 8: Net-(R8-Pad2) -> unconnected-(U4-Pad8)
- U4 pad 9: Net-(R8-Pad1) -> unconnected-(U4-Pad9)
- U6 pad 5: Net-(U4-Pad3) -> Net-(TP9-Pad1)

Commit message: wip layout (5)
Parts:
- moved TP8 173.4 mm to (76.3, 101.5), turned to 180 degrees
- moved R16 165.2 mm to (84.5, 188.2), turned to 90 degrees
- moved D12 159.2 mm to (91.3, 182.2), turned to 90 degrees
- moved D9 155.7 mm to (79.8, 183.6), turned to 90 degrees
- moved R13 153.7 mm to (73.9, 189.4), turned to 90 degrees
- moved D11 137.4 mm to (87.5, 181.7), turned to 90 degrees
- moved D8 129.1 mm to (77.2, 184.7), turned to 90 degrees
- moved R17 128.0 mm to (87.6, 188.5), turned to 90 degrees
- moved R1 125.5 mm to (102.1, 28.5)
- moved D7 123.3 mm to (73.7, 184.0), turned to 90 degrees
- moved Ct1 119.5 mm to (85.0, 91.2), turned to 180 degrees
- moved C5 118.5 mm to (88.8, 81.8)
- moved C3 117.4 mm to (85.7, 78.5), turned to 90 degrees
- moved C13 115.3 mm to (78.7, 78.5)
- moved C4 114.1 mm to (88.8, 79.8)
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
Commit message: wip layout (6)
Parts:
- moved C7 135.6 mm to (62.0, 74.4), turned to 180 degrees
- moved R18 132.8 mm to (118.9, 58.3), turned to 0 degrees
- moved TP8 126.2 mm to (196.4, 140.1)
- moved D12 124.8 mm to (118.9, 60.5), turned to 0 degrees
- moved R13 108.6 mm to (49.0, 83.7), turned to 0 degrees
- moved D7 101.4 mm to (49.0, 85.7), turned to 0 degrees
- moved R17 84.8 mm to (73.0, 105.0), turned to 180 degrees
- moved R16 81.0 mm to (73.0, 108.0), turned to 180 degrees
- moved D11 78.9 mm to (69.0, 105.0), turned to 0 degrees
- moved R15 78.0 mm to (73.0, 111.0), turned to 180 degrees
- moved D10 76.3 mm to (69.0, 108.0), turned to 0 degrees
- moved R14 75.3 mm to (72.9, 114.0), turned to 180 degrees
- moved D9 73.4 mm to (69.0, 111.0), turned to 0 degrees
- moved D8 71.2 mm to (69.0, 114.0), turned to 0 degrees
- moved R11 59.5 mm to (86.4, 112.3), turned to -90 degrees
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
Commit message: wip layout (7)
Parts:
- moved TP8 71.1 mm to (144.0, 92.0), turned to -90 degrees
- moved Ct1 3.98 mm to (88.5, 89.5), turned to 0 degrees
- moved R11 3.97 mm to (83.3, 109.8)
- moved A1 3.97 mm to (118.8, 92.9)
- moved D10 3.97 mm to (65.9, 105.5)
- moved D11 3.97 mm to (65.9, 102.5)
- moved D8 3.97 mm to (65.9, 111.5)
- moved D9 3.97 mm to (65.9, 108.5)
- moved R10 3.97 mm to (80.7, 109.8)
- moved R14 3.97 mm to (69.8, 111.5)
- moved R15 3.97 mm to (69.9, 108.5)
- moved R16 3.97 mm to (69.9, 105.5)
- moved R17 3.97 mm to (69.9, 102.5)
- moved TP1 2.00 mm to (66.0, 34.0)
- moved Rt1 0.30 mm to (85.0, 89.5)
Other:
- board outline added: 90 x 90 mm
Changed lines of the file:
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@@
   (net 71 "unconnected-(U4-Pad10)")
   (footprint "Resistor_SMD:R_0805_2012Metric" (layer "F.Cu")
-    (at 83.8 112.3 -90)
+    (at 80.7 109.8125 -90)
     (descr "Resistor SMD 0805 (2012 Metric), square (rectangular) end terminal, IPC_7351 nominal, (Body size source: IPC-SM-782 page 72, https://www.pcb-3d.com/wordpress/wp-content/uploads/ipc-sm-782a_amendment_1_and_2.pdf), generated with kicad-footprint-generator")
     (tags "resistor")
@@
   )
   (footprint "LED_SMD:LED_0603_1608Metric" (layer "F.Cu")
-    (at 69 105)
+    (at 65.9 102.5125)
     (descr "LED SMD 0603 (1608 Metric), square (rectangular) end terminal, IPC_7351 nominal, (Body size source: http://www.tortai-tech.com/upload/download/2011102023233369053.pdf), generated with kicad-footprint-generator")
     (tags "LED")
@@
   )
   (footprint "Resistor_SMD:R_0805_2012Metric" (layer "F.Cu")
-    (at 72.9125 114 180)
+    (at 69.8125 111.5125 180)
     (descr "Resistor SMD 0805 (2012 Metric), square (rectangular) end terminal, IPC_7351 nominal, (Body size source: IPC-SM-782 page 72, https://www.pcb-3d.com/wordpress/wp-content/uploads/ipc-sm-782a_amendment_1_and_2.pdf), generated with kicad-footprint-generator")
     (tags "resistor")
@@
   )
   (footprint "LED_SMD:LED_0603_1608Metric" (layer "F.Cu")
-    (at 69 111)
+    (at 65.9 108.5125)
     (descr "LED SMD 0603 (1608 Metric), square (rectangular) end terminal, IPC_7351 nominal, (Body size source: http://www.tortai-tech.com/upload/download/2011102023233369053.pdf), generated with kicad-footprint-generator")
     (tags "LED")
@@
   )
   (footprint "LED_SMD:LED_0603_1608Metric" (layer "F.Cu")
-    (at 69 114)
+    (at 65.9 111.5125)
     (descr "LED SMD 0603 (1608 Metric), square (rectangular) end terminal, IPC_7351 nominal, (Body size source: http://www.tortai-tech.com/upload/download/2011102023233369053.pdf), generated with kicad-footprint-generator")
     (tags "LED")
@@
   )
   (footprint "small_wind_turbine:Oscilloscope_Test_Point" (layer "F.Cu")
-    (at 66 32)
+    (at 66 34)
     (descr "Keystone Miniature THM Test Point 5010-5014, http://www.keyelco.com/product-pdf.cfm?p=1319")
     (tags "Through Hole Mount Test Points")
@@
   )
   (footprint "Resistor_SMD:R_0805_2012Metric" (layer "F.Cu")
-    (at 84.9875 89.2)
+    (at 84.9875 89.5)
     (descr "Resistor SMD 0805 (2012 Metric), square (rectangular) end terminal, IPC_7351 nominal, (Body size source: IPC-SM-782 page 72, https://www.pcb-3d.com/wordpress/wp-content/uploads/ipc-sm-782a_amendment_1_and_2.pdf), generated with kicad-footprint-generator")
     (tags "resistor")
@@
   )
   (footprint "Resistor_SMD:R_0805_2012Metric" (layer "F.Cu")
-    (at 73 105 180)
+    (at 69.9 102.5125 180)
     (descr "Resistor SMD 0805 (2012 Metric), square (rectangular) end terminal, IPC_7351 nominal, (Body size source: IPC-SM-782 page 72, https://www.pcb-3d.com/wordpress/wp-content/uploads/ipc-sm-782a_amendment_1_and_2.pdf), generated with kicad-footprint-generator")
     (tags "resistor")
@@
   )
   (footprint "Resistor_SMD:R_0805_2012Metric" (layer "F.Cu")
-    (at 86.4 112.2875 -90)
+    (at 83.3 109.8 -90)
     (descr "Resistor SMD 0805 (2012 Metric), square (rectangular) end terminal, IPC_7351 nominal, (Body size source: IPC-SM-782 page 72, https://www.pcb-3d.com/wordpress/wp-content/uploads/ipc-sm-782a_amendment_1_and_2.pdf), generated with kicad-footprint-generator")
     (tags "resistor")
@@
   )
   (footprint "small_wind_turbine:Oscilloscope_Test_Point" (layer "F.Cu")
-    (at 196.4 140.1 180)
+    (at 144 92 -90)
     (descr "Keystone Miniature THM Test Point 5010-5014, http://www.keyelco.com/product-pdf.cfm?p=1319")
     (tags "Through Hole Mount Test Points")
@@
     (property "Sheetname" "")
     (attr through_hole)
-    (fp_text reference "TP8" (at 0 -2.75) (layer "F.SilkS")
+    (fp_text reference "TP8" (at 0 -2.75 90) (layer "F.SilkS")
       (effects (font (size 1 1) (thickness 0.15)))
     )
-    (fp_text value "TestPoint_2Pole" (at 0 2.75) (layer "F.Fab")
+    (fp_text value "TestPoint_2Pole" (at 0 2.75 90) (layer "F.Fab")
       (effects (font (size 1 1) (thickness 0.15)))
     )
-    (fp_text user "${REFERENCE}" (at 0 0) (layer "F.Fab")
+    (fp_text user "${REFERENCE}" (at 0 0 90) (layer "F.Fab")
       (effects (font (size 0.6 0.6) (thickness 0.09)))
     )
@@
     (fp_line (start 1.25 -0.4) (end 1.25 0.4) (layer "F.Fab") (width 0.15))
     (fp_circle (center 0 0) (end 1.6 0) (layer "F.Fab") (width 0.15) (fill none))
-    (pad "1" thru_hole circle (at 0 0 180) (size 2.8 2.8) (drill 1.6) (layers *.Cu *.Mask)
+    (pad "1" thru_hole circle (at 0 0 270) (size 2.8 2.8) (drill 1.6) (layers *.Cu *.Mask)
       (net 29 "Net-(Cbs1-Pad1)") (pinfunction "1") (pintype "passive"))
-    (pad "2" thru_hole circle (at 5 0 180) (size 2.5 2.5) (drill 1.2) (layers *.Cu *.Mask)
+    (pad "2" thru_hole circle (at 5 0 270) (size 2.5 2.5) (drill 1.2) (layers *.Cu *.Mask)
       (net 4 "GND") (pinfunction "2") (pintype "passive"))
-    (pad "2" thru_hole circle (at -5 0 180) (size 2.5 2.5) (drill 1.2) (layers *.Cu *.Mask)
+    (pad "2" thru_hole circle (at -5 0 270) (size 2.5 2.5) (drill 1.2) (layers *.Cu *.Mask)
       (net 4 "GND") (pinfunction "2") (pintype "passive"))
     (model "${KICAD6_3DMODEL_DIR}/TestPoint.3dshapes/TestPoint_Keystone_5010-5014_Multipurpose.wrl"
@@
   )
   (footprint "Module:Adafruit_Feather" (layer "F.Cu")
-    (at 121.85 95.435 -90)
+    (at 118.75 92.9475 -90)
     (descr "Common footprint for the Adafruit Feather series of boards, https://learn.adafruit.com/adafruit-feather/feather-specification")
     (tags "Adafruit Feather")
@@
   )
   (footprint "Capacitor_SMD:C_0805_2012Metric" (layer "F.Cu")
-    (at 84.95 91.2 180)
+    (at 88.55 89.5)
     (descr "Capacitor SMD 0805 (2012 Metric), square (rectangular) end terminal, IPC_7351 nominal, (Body size source: IPC-SM-782 page 76, https://www.pcb-3d.com/wordpress/wp-content/uploads/ipc-sm-782a_amendment_1_and_2.pdf, https://docs.google.com/spreadsheets/d/1BsfQQcO9C6DZCsRaXUlFlo91Tg2WpOkGARC1WS5S8t0/edit?usp=sharing), generated with kicad-footprint-generator")
     (tags "capacitor")
@@
     (fp_line (start 1 -0.625) (end 1 0.625) (layer "F.Fab") (width 0.1))
     (fp_line (start -1 -0.625) (end 1 -0.625) (layer "F.Fab") (width 0.1))
-    (pad "1" smd roundrect (at -0.95 0 180) (size 1 1.45) (layers "F.Cu" "F.Paste" "F.Mask") (roundrect_rratio 0.25)
+    (pad "1" smd roundrect (at -0.95 0) (size 1 1.45) (layers "F.Cu" "F.Paste" "F.Mask") (roundrect_rratio 0.25)
       (net 35 "Net-(Ct1-Pad1)") (pintype "passive"))
-    (pad "2" smd roundrect (at 0.95 0 180) (size 1 1.45) (layers "F.Cu" "F.Paste" "F.Mask") (roundrect_rratio 0.25)
+    (pad "2" smd roundrect (at 0.95 0) (size 1 1.45) (layers "F.Cu" "F.Paste" "F.Mask") (roundrect_rratio 0.25)
       (net 4 "GND") (pintype "passive"))
     (model "${KICAD6_3DMODEL_DIR}/Capacitor_SMD.3dshapes/C_0805_2012Metric.wrl"
@@
   )
   (footprint "Resistor_SMD:R_0805_2012Metric" (layer "F.Cu")
-    (at 73 108 180)
+    (at 69.9 105.5125 180)
     (descr "Resistor SMD 0805 (2012 Metric), square (rectangular) end terminal, IPC_7351 nominal, (Body size source: IPC-SM-782 page 72, https://www.pcb-3d.com/wordpress/wp-content/uploads/ipc-sm-782a_amendment_1_and_2.pdf), generated with kicad-footprint-generator")
     (tags "resistor")
@@
   )
   (footprint "Resistor_SMD:R_0805_2012Metric" (layer "F.Cu")
-    (at 73 111 180)
+    (at 69.9 108.5125 180)
     (descr "Resistor SMD 0805 (2012 Metric), square (rectangular) end terminal, IPC_7351 nominal, (Body size source: IPC-SM-782 page 72, https://www.pcb-3d.com/wordpress/wp-content/uploads/ipc-sm-782a_amendment_1_and_2.pdf), generated with kicad-footprint-generator")
     (tags "resistor")
@@
   )
   (footprint "LED_SMD:LED_0603_1608Metric" (layer "F.Cu")
-    (at 69 108)
+    (at 65.9 105.5125)
     (descr "LED SMD 0603 (1608 Metric), square (rectangular) end terminal, IPC_7351 nominal, (Body size source: http://www.tortai-tech.com/upload/download/2011102023233369053.pdf), generated with kicad-footprint-generator")
     (tags "LED")
@@
   (gr_line (start 77 69) (end 71 69) (layer "Cmts.User") (width 0.15))
   (gr_line (start 50 41) (end 63 39) (layer "Cmts.User") (width 0.15))
+  (gr_line (start 131 31) (end 131 121) (layer "Edge.Cuts") (width 0.1))
+  (gr_line (start 131 121) (end 41 121) (layer "Edge.Cuts") (width 0.1))
+  (gr_line (start 41 31) (end 131 31) (layer "Edge.Cuts") (width 0.1))
+  (gr_line (start 41 121) (end 41 31) (layer "Edge.Cuts") (width 0.1))
 )
